Commit message: realsense plugin is ok

File: src/robots/go2_description/xacro/_d435i.gazebo.xacro (robot description, xacro)
@@ -197,7 +197,7 @@
                 <infrared2OpticalframeName>${infrared2_optical_frame}</infrared2OpticalframeName>
                 <!-- Depth camera settings -->
-                <rangeMinDepth>0.2</rangeMinDepth>
+                <rangeMinDepth>0.1</rangeMinDepth>
                 <xacro:unless value="${clip_distance > 0.0}">
-                    <rangeMaxDepth>10.0</rangeMaxDepth>
+                    <rangeMaxDepth>2.0</rangeMaxDepth>
                 </xacro:unless>
                 <xacro:if value="${clip_distance > 0.0}">

File: src/robots/go2_description/xacro/_d435i.urdf.xacro (robot description, xacro)
@@ -37,5 +37,5 @@
                                           topics_ns:=camera
                                           visualize:=true
-                                          align_depth:=false
+                                          align_depth:=true
                                           enable_pointCloud:=true
                                           unite_imu_method:=linear_interpolation

File: src/robots/go2_description/xacro/robot.xacro (robot description, xacro)
@@ -8,4 +8,5 @@
     <xacro:include filename="$(find go2_description)/xacro/gazebo.xacro"/>
     <xacro:include filename="$(find a1_description)/xacro/ros2_control.xacro"/>
+    <xacro:include filename="$(find go2_description)/xacro/_d435i.urdf.xacro"/>
     <!-- <xacro:include filename="$(find go2_gazebo)/launch/stairs.urdf.xacro"/> -->
     <!-- <xacro:stairs stairs="15" xpos="0" ypos="0" zpos="0" /> -->
@@ -112,3 +113,7 @@
     <xacro:leg name="RR" mirror="-1" mirror_dae="False"  front_hind="-1" front_hind_dae="False" />
     <xacro:leg name="RL" mirror="1"  mirror_dae="True"   front_hind="-1" front_hind_dae="False" />
+    <!-- D345i相机 -->
+    <xacro:sensor_d435i parent="trunk" name="camera" topics_ns="camera">
+        <origin  xyz="0.345 0 0.07" rpy="0 0.25 0"/>
+    </xacro:sensor_d435i>
 </robot>
