Commit message: can run but policy some problem

File: src/robots/go2_description/xacro/robot.xacro (robot description, xacro)
@@ -3,3 +3,8 @@
     <xacro:include filename="$(find go2_description)/urdf/go2_description.urdf"/>
     <xacro:include filename="$(find go2_description)/xacro/gazebo.xacro"/>
+    <!-- D34i相机 -->
+    <xacro:include filename="$(find go2w_description)/xacro/_d435i.urdf.xacro"/>
+    <xacro:sensor_d435i parent="base" name="camera" topics_ns="camera">
+        <origin  xyz="0.345 0 0.07" rpy="0 0.25 0"/>
+    </xacro:sensor_d435i>
 </robot>

Commit message: can run

File: src/robots/go2_description/xacro/robot.xacro (robot description, xacro)
@@ -6,5 +6,5 @@
     <xacro:include filename="$(find go2w_description)/xacro/_d435i.urdf.xacro"/>
     <xacro:sensor_d435i parent="base" name="camera" topics_ns="camera">
-        <origin  xyz="0.345 0 0.07" rpy="0 0.25 0"/>
+        <origin  xyz="0.25489 0.0 0.05999" rpy="0 0.25 0"/>
     </xacro:sensor_d435i>
 </robot>

Commit message: can run version

File: src/robots/go2_description/xacro/robot.xacro (robot description, xacro)
@@ -4,5 +4,5 @@
     <xacro:include filename="$(find go2_description)/xacro/gazebo.xacro"/>
     <!-- D34i相机 -->
-    <xacro:include filename="$(find go2w_description)/xacro/_d435i.urdf.xacro"/>
+    <xacro:include filename="$(find go2_description)/xacro/_d435i.urdf.xacro"/>
     <xacro:sensor_d435i parent="base" name="camera" topics_ns="camera">
         <origin  xyz="0.25489 0.0 0.05999" rpy="0 0.25 0"/>

File: src/robots/lite3_description/urdf/lite3.urdf (robot description, URDF)
Before this commit: robot Lite3, 19 links, 18 joints
Links:
- removed link INERTIA
- removed link MODULE
- added link imu_link, mass 0
- link FL_FOOT: mass 0.08 -> 0.02; geometry collision sphere radius=0.022; visual sphere radius=0.022
- link FL_HIP: geometry collision cylinder length=0.15 radius=0.04; visual mesh filename=package://lite3_description/meshes/fl_hip.STL
- link FL_SHANK: mass 0.1729 -> 0.153; geometry collision cylinder length=0.10 radius=0.015; collision cylinder length=0.12 radius=0.015
- link FL_THIGH: geometry collision box size=0.04 0.045 0.2; visual mesh filename=package://lite3_description/meshes/fl_thigh.STL
- link FR_FOOT: mass 0.08 -> 0.02; geometry collision sphere radius=0.022; visual sphere radius=0.022
- link FR_HIP: geometry collision cylinder length=0.15 radius=0.04; visual mesh filename=package://lite3_description/meshes/fr_hip.STL
- link FR_SHANK: mass 0.1729 -> 0.153; geometry collision cylinder length=0.10 radius=0.015; collision cylinder length=0.12 radius=0.015
- link FR_THIGH: geometry collision box size=0.04 0.045 0.2; visual mesh filename=package://lite3_description/meshes/fr_thigh.STL
- link HL_FOOT: mass 0.08 -> 0.02; geometry collision sphere radius=0.022; visual sphere radius=0.022
- link HL_HIP: geometry collision cylinder length=0.15 radius=0.04; visual mesh filename=package://lite3_description/meshes/hl_hip.STL
- link HL_SHANK: mass 0.1729 -> 0.153; geometry collision cylinder length=0.10 radius=0.015; collision cylinder length=0.12 radius=0.015
- link HL_THIGH: geometry collision box size=0.04 0.045 0.2; visual mesh filename=package://lite3_description/meshes/hl_thigh.STL
- link HR_FOOT: mass 0.08 -> 0.02; geometry collision sphere radius=0.022; visual sphere radius=0.022
- link HR_HIP: geometry collision cylinder length=0.15 radius=0.04; visual mesh filename=package://lite3_description/meshes/hr_hip.STL
- link HR_SHANK: mass 0.1729 -> 0.153; geometry collision cylinder length=0.10 radius=0.015; collision cylinder length=0.12 radius=0.015
- link HR_THIGH: geometry collision box size=0.04 0.045 0.2; visual mesh filename=package://lite3_description/meshes/hr_thigh.STL
- link TORSO: mass None -> 5.6056; geometry collision box size=0.25 0.2 0.12; collision box size=0.5 0.1 0.12
Joints:
- removed joint Torso2Inertia
- removed joint Torso2MODULE
- added joint imu_joint: type fixed, parent TORSO, child imu_link, origin xyz=-0.02557 0 0.04232 rpy=0 0 0, axis 0 0 0
- joint FL_HipX_joint: axis 1 0 0 -> -1 0 0; limit lower=-0.523 upper=0.523 effort=21 velocity=23.5 -> lower=-0.523 upper=0.523 effort=24 velocity=26.2; origin xyz=0.1745 -0.062 0 -> xyz=0.1745 0.062 0 rpy=0 0 0
- joint FL_HipY_joint: axis 0 1 0 -> 0 -1 0; limit lower=-0.314 upper=2.67 effort=21 velocity=23 -> lower=-2.67 upper=0.314 effort=24 velocity=26.2; origin xyz=0 -0.09735 0 -> xyz=0 0.09735 0 rpy=0 0 0
- joint FL_Knee_joint: axis 0 1 0 -> 0 -1 0; limit lower=-2.792 upper=-0.524 effort=32 velocity=18.21 -> lower=0.524 upper=2.792 effort=36 velocity=17.3; origin xyz=0 0 -0.20 -> xyz=0 0 -0.20 rpy=0 0 0
- joint FR_HipX_joint: axis 1 0 0 -> -1 0 0; limit lower=-0.523 upper=0.523 effort=21 velocity=23.5 -> lower=-0.523 upper=0.523 effort=24 velocity=26.2; origin xyz=0.1745 0.062 0 -> xyz=0.1745 -0.062 0 rpy=0 0 0
- joint FR_HipY_joint: axis 0 1 0 -> 0 -1 0; limit lower=-0.314 upper=2.67 effort=21 velocity=23 -> lower=-2.67 upper=0.314 effort=24 velocity=26.2; origin xyz=0 0.09735 0 -> xyz=0 -0.09735 0 rpy=0 0 0
- joint FR_Knee_joint: axis 0 1 0 -> 0 -1 0; limit lower=-2.792 upper=-0.524 effort=32 velocity=18.21 -> lower=0.524 upper=2.792 effort=36 velocity=17.3; origin xyz=0 0 -0.20 -> xyz=0 0 -0.20 rpy=0 0 0
- joint HL_HipX_joint: axis 1 0 0 -> -1 0 0; limit lower=-0.523 upper=0.523 effort=21 velocity=23.5 -> lower=-0.523 upper=0.523 effort=24 velocity=26.2; origin xyz=-0.1745 -0.062 0 -> xyz=-0.1745 0.062 0 rpy=0 0 0
- joint HL_HipY_joint: axis 0 1 0 -> 0 -1 0; limit lower=-0.314 upper=2.67 effort=21 velocity=23 -> lower=-2.67 upper=0.314 effort=24 velocity=26.2; origin xyz=0 -0.09735 0 -> xyz=0 0.09735 0 rpy=0 0 0
- joint HL_Knee_joint: axis 0 1 0 -> 0 -1 0; limit lower=-2.792 upper=-0.524 effort=32 velocity=18.21 -> lower=0.524 upper=2.792 effort=36 velocity=17.3; origin xyz=0 0 -0.20 -> xyz=0 0 -0.20 rpy=0 0 0
- joint HR_HipX_joint: axis 1 0 0 -> -1 0 0; limit lower=-0.523 upper=0.523 effort=21 velocity=23.5 -> lower=-0.523 upper=0.523 effort=24 velocity=26.2; origin xyz=-0.1745 0.062 0 -> xyz=-0.1745 -0.062 0 rpy=0 0 0
- joint HR_HipY_joint: axis 0 1 0 -> 0 -1 0; limit lower=-0.314 upper=2.67 effort=21 velocity=23 -> lower=-2.67 upper=0.314 effort=24 velocity=26.2; origin xyz=0 0.09735 0 -> xyz=0 -0.09735 0 rpy=0 0 0
- joint HR_Knee_joint: axis 0 1 0 -> 0 -1 0; limit lower=-2.792 upper=-0.524 effort=32 velocity=18.21 -> lower=0.524 upper=2.792 effort=36 velocity=17.3; origin xyz=0 0 -0.20 -> xyz=0 0 -0.20 rpy=0 0 0

File: src/robots/lite3_description/xacro/_d435i.gazebo.xacro (robot description, xacro)
@@ -25,7 +25,7 @@
                                             gyro_fps:=400
                                             clip_distance:=-1.0
-                                            near_clip:=0.01
-                                            range_min_depth:=0.01
-                                            pointcloud_cutoff:=0.01
+                                            near_clip:=0.001
+                                            range_min_depth:=0.001
+                                            pointcloud_cutoff:=0.001
                                             depth_width:=1280
                                             depth_height:=720

File: src/robots/lite3_description/xacro/robot.xacro (robot description, xacro)
@@ -3,8 +3,8 @@
     <xacro:include filename="$(find lite3_description)/urdf/lite3.urdf"/>
     <xacro:include filename="$(find lite3_description)/xacro/gazebo.xacro"/>
-    <!-- D34i相机 -->
-    <xacro:include filename="$(find lite3_description)/xacro/_d435i.urdf.xacro"/>
-    <xacro:sensor_d435i parent="TORSO" name="camera" topics_ns="camera">
-        <origin  xyz="0.25489 0.0175 0.07249" rpy="0 0.25 0"/>
-    </xacro:sensor_d435i>
+     <!-- D34i相机 -->
+     <xacro:include filename="$(find lite3_description)/xacro/_d435i.urdf.xacro"/>
+     <xacro:sensor_d435i parent="TORSO" name="camera" topics_ns="camera">
+         <origin  xyz="0.25489 0.0 0.05999" rpy="0 0.25 0"/>
+     </xacro:sensor_d435i>
 </robot>
