Commit message: debug

File: src/robots/go2w_description/xacro/robot.xacro (robot description, xacro)
@@ -3,3 +3,8 @@
     <xacro:include filename="$(find go2w_description)/urdf/go2w_description.urdf"/>
     <xacro:include filename="$(find go2w_description)/xacro/gazebo.xacro"/>
+     <!-- D34i相机 -->
+     <xacro:include filename="$(find go2w_description)/xacro/_d435i.urdf.xacro"/>
+     <xacro:sensor_d435i parent="base" name="camera" topics_ns="camera">
+         <origin  xyz="0.345 0 0.07" rpy="0 0.25 0"/>
+     </xacro:sensor_d435i>
 </robot>
