Commit message: add lite3

File: src/robots/lite3_description/urdf/lite3.urdf (robot description, URDF)
Before this commit: robot Lite3, 18 links, 17 joints
Links:
- removed link imu_link
- added link INERTIA, mass 7.530
- link FL_FOOT: mass 0.02 -> 0.08; geometry collision sphere radius=0.023
- link FL_HIP: mass 0.550 -> 0.428; geometry visual mesh filename=package://lite3_description/meshes/FL_HIP.dae
- link FL_SHANK: mass 0.153 -> 0.115; geometry collision box size=0.02 0.02 0.23; visual mesh filename=package://lite3_description/meshes/SHANK.dae
- link FL_THIGH: mass 0.86 -> 0.61; geometry collision box size=0.035 0.035 0.218; collision cylinder length=0.05 radius=0.042
- link FR_FOOT: mass 0.02 -> 0.08; geometry collision sphere radius=0.023
- link FR_HIP: mass 0.550 -> 0.428; geometry visual mesh filename=package://lite3_description/meshes/FR_HIP.dae
- link FR_SHANK: mass 0.153 -> 0.115; geometry collision box size=0.02 0.02 0.23; visual mesh filename=package://lite3_description/meshes/SHANK.dae
- link FR_THIGH: mass 0.86 -> 0.61; geometry collision box size=0.035 0.035 0.218; collision cylinder length=0.05 radius=0.042
- link HL_FOOT: mass 0.02 -> 0.08; geometry collision sphere radius=0.023
- link HL_HIP: mass 0.550 -> 0.428; geometry visual mesh filename=package://lite3_description/meshes/HL_HIP.dae
- link HL_SHANK: mass 0.153 -> 0.115; geometry collision box size=0.02 0.02 0.23; visual mesh filename=package://lite3_description/meshes/SHANK.dae
- link HL_THIGH: mass 0.86 -> 0.61; geometry collision box size=0.035 0.035 0.218; collision cylinder length=0.05 radius=0.042
- link HR_FOOT: mass 0.02 -> 0.08; geometry collision sphere radius=0.023
- link HR_HIP: mass 0.550 -> 0.428; geometry visual mesh filename=package://lite3_description/meshes/HR_HIP.dae
- link HR_SHANK: mass 0.153 -> 0.115; geometry collision box size=0.02 0.02 0.23; visual mesh filename=package://lite3_description/meshes/SHANK.dae
- link HR_THIGH: mass 0.86 -> 0.61; geometry collision box size=0.035 0.035 0.218; collision cylinder length=0.05 radius=0.042
- link TORSO: mass 5.6056 -> None; geometry collision box size=0.42 0.12 0.08; visual mesh filename=package://lite3_description/meshes/Lite3.dae
Joints:
- removed joint imu_joint
- added joint Torso2Inertia: type fixed, parent TORSO, child INERTIA
- joint FL_Ankle: origin xyz=0 0 -0.21012 -> xyz=-0.007 0 -0.21
- joint FL_HipX_joint: axis -1 0 0 -> 1 0 0; limit lower=-0.523 upper=0.523 effort=24 velocity=26.2 -> lower=-0.523 upper=0.523 effort=21 velocity=23.5; origin xyz=0.1745 0.062 0 rpy=0 0 0 -> xyz=0.1245 -0.062 0
- joint FL_HipY_joint: axis 0 -1 0 -> 0 1 0; limit lower=-2.67 upper=0.314 effort=24 velocity=26.2 -> lower=-0.314 upper=2.67 effort=21 velocity=23; origin xyz=0 0.09735 0 rpy=0 0 0 -> xyz=0 -0.0985 0
- joint FL_Knee_joint: axis 0 -1 0 -> 0 1 0; limit lower=0.524 upper=2.792 effort=36 velocity=17.3 -> lower=-2.792 upper=-0.524 effort=32 velocity=18.21; origin xyz=0 0 -0.20 rpy=0 0 0 -> xyz=0 0 -0.20
- joint FR_Ankle: origin xyz=0 0 -0.21012 -> xyz=-0.007 0 -0.21
- joint FR_HipX_joint: axis -1 0 0 -> 1 0 0; limit lower=-0.523 upper=0.523 effort=24 velocity=26.2 -> lower=-0.523 upper=0.523 effort=21 velocity=23.5; origin xyz=0.1745 -0.062 0 rpy=0 0 0 -> xyz=0.1245 0.062 0
- joint FR_HipY_joint: axis 0 -1 0 -> 0 1 0; limit lower=-2.67 upper=0.314 effort=24 velocity=26.2 -> lower=-0.314 upper=2.67 effort=21 velocity=23; origin xyz=0 -0.09735 0 rpy=0 0 0 -> xyz=0 0.0985 0
- joint FR_Knee_joint: axis 0 -1 0 -> 0 1 0; limit lower=0.524 upper=2.792 effort=36 velocity=17.3 -> lower=-2.792 upper=-0.524 effort=32 velocity=18.21; origin xyz=0 0 -0.20 rpy=0 0 0 -> xyz=0 0 -0.20
- joint HL_Ankle: origin xyz=0 0 -0.21012 -> xyz=-0.007 0 -0.21
- joint HL_HipX_joint: axis -1 0 0 -> 1 0 0; limit lower=-0.523 upper=0.523 effort=24 velocity=26.2 -> lower=-0.523 upper=0.523 effort=21 velocity=23.5; origin xyz=-0.1745 0.062 0 rpy=0 0 0 -> xyz=-0.2245 -0.062 0
- joint HL_HipY_joint: axis 0 -1 0 -> 0 1 0; limit lower=-2.67 upper=0.314 effort=24 velocity=26.2 -> lower=-0.314 upper=2.67 effort=21 velocity=23; origin xyz=0 0.09735 0 rpy=0 0 0 -> xyz=0 -0.0985 0
- joint HL_Knee_joint: axis 0 -1 0 -> 0 1 0; limit lower=0.524 upper=2.792 effort=36 velocity=17.3 -> lower=-2.792 upper=-0.524 effort=32 velocity=18.21; origin xyz=0 0 -0.20 rpy=0 0 0 -> xyz=0 0 -0.20
- joint HR_Ankle: origin xyz=0 0 -0.21012 -> xyz=-0.007 0 -0.21
- joint HR_HipX_joint: axis -1 0 0 -> 1 0 0; limit lower=-0.523 upper=0.523 effort=24 velocity=26.2 -> lower=-0.523 upper=0.523 effort=21 velocity=23.5; origin xyz=-0.1745 -0.062 0 rpy=0 0 0 -> xyz=-0.2245 0.062 0
- joint HR_HipY_joint: axis 0 -1 0 -> 0 1 0; limit lower=-2.67 upper=0.314 effort=24 velocity=26.2 -> lower=-0.314 upper=2.67 effort=21 velocity=23; origin xyz=0 -0.09735 0 rpy=0 0 0 -> xyz=0 0.0985 0
- joint HR_Knee_joint: axis 0 -1 0 -> 0 1 0; limit lower=0.524 upper=2.792 effort=36 velocity=17.3 -> lower=-2.792 upper=-0.524 effort=32 velocity=18.21; origin xyz=0 0 -0.20 rpy=0 0 0 -> xyz=0 0 -0.20

File: src/robots/lite3_description/xacro/robot.xacro (robot description, xacro)
@@ -3,3 +3,8 @@
     <xacro:include filename="$(find lite3_description)/urdf/lite3.urdf"/>
     <xacro:include filename="$(find lite3_description)/xacro/gazebo.xacro"/>
+    <!-- D34i相机 -->
+    <xacro:include filename="$(find lite3_description)/xacro/_d435i.urdf.xacro"/>
+    <xacro:sensor_d435i parent="TORSO" name="camera" topics_ns="camera">
+        <origin  xyz="0.345 0 0.07" rpy="0 0.25 0"/>
+    </xacro:sensor_d435i>
 </robot>

Commit message: lite3

File: src/robots/lite3_description/urdf/lite3.urdf (robot description, URDF)
Before this commit: robot Lite3, 18 links, 17 joints
Links:
- added link MODULE, mass 0.8835; collision box size=0.4 0.12 0.05064
- link FL_HIP: mass 0.428 -> 0.550
- link FL_SHANK: mass 0.115 -> 0.1729
- link FL_THIGH: mass 0.61 -> 0.86; geometry collision box size=0.035 0.035 0.215; collision cylinder length=0.05 radius=0.042
- link FR_HIP: mass 0.428 -> 0.550
- link FR_SHANK: mass 0.115 -> 0.1729
- link FR_THIGH: mass 0.61 -> 0.86; geometry collision box size=0.035 0.035 0.215; collision cylinder length=0.05 radius=0.042
- link HL_HIP: mass 0.428 -> 0.550
- link HL_SHANK: mass 0.115 -> 0.1729
- link HL_THIGH: mass 0.61 -> 0.86; geometry collision box size=0.035 0.035 0.215; collision cylinder length=0.05 radius=0.042
- link HR_HIP: mass 0.428 -> 0.550
- link HR_SHANK: mass 0.115 -> 0.1729
- link HR_THIGH: mass 0.61 -> 0.86; geometry collision box size=0.035 0.035 0.215; collision cylinder length=0.05 radius=0.042
- link INERTIA: mass 7.530 -> 6.16956
- link TORSO: geometry collision box size=0.44 0.12 0.09786; visual mesh filename=package://lite3_description/meshes/Lite3.dae
Joints:
- added joint Torso2MODULE: type fixed, parent TORSO, child MODULE
- joint FL_Ankle: origin xyz=-0.007 0 -0.21 -> xyz=0 0 -0.21012
- joint FL_HipX_joint: origin xyz=0.1245 -0.062 0 -> xyz=0.1745 -0.062 0
- joint FL_HipY_joint: origin xyz=0 -0.0985 0 -> xyz=0 -0.09735 0
- joint FR_Ankle: origin xyz=-0.007 0 -0.21 -> xyz=0 0 -0.21012
- joint FR_HipX_joint: origin xyz=0.1245 0.062 0 -> xyz=0.1745 0.062 0
- joint FR_HipY_joint: origin xyz=0 0.0985 0 -> xyz=0 0.09735 0
- joint HL_Ankle: origin xyz=-0.007 0 -0.21 -> xyz=0 0 -0.21012
- joint HL_HipX_joint: origin xyz=-0.2245 -0.062 0 -> xyz=-0.1745 -0.062 0
- joint HL_HipY_joint: origin xyz=0 -0.0985 0 -> xyz=0 -0.09735 0
- joint HR_Ankle: origin xyz=-0.007 0 -0.21 -> xyz=0 0 -0.21012
- joint HR_HipX_joint: origin xyz=-0.2245 0.062 0 -> xyz=-0.1745 0.062 0
- joint HR_HipY_joint: origin xyz=0 0.0985 0 -> xyz=0 0.09735 0

File: src/robots/lite3_description/xacro/robot.xacro (robot description, xacro)
@@ -6,5 +6,5 @@
     <xacro:include filename="$(find lite3_description)/xacro/_d435i.urdf.xacro"/>
     <xacro:sensor_d435i parent="TORSO" name="camera" topics_ns="camera">
-        <origin  xyz="0.345 0 0.07" rpy="0 0.25 0"/>
+        <origin  xyz="0.25489 0.0175 0.07249" rpy="0 0.25 0"/>
     </xacro:sensor_d435i>
 </robot>
